File: usb-pd-splitter.kicad_sch (KiCad schematic)
At the start: 3 parts, among them J1 USB_C_Receptacle_USB2.0_14P, J2 USB_C_Receptacle_USB2.0_14P, J3 USB_C_Receptacle_USB2.0_14P

Commit message: schematic done
Parts:
- added R1, R2: 5.1k, Resistor_SMD:R_0805_2012Metric_Pad1.20x1.40mm_HandSolder, symbol Device:R_US
- J1, J2, J3: footprint (none) -> Connector_USB:USB_C_Receptacle_GCT_USB4110
Connections:
- net GND: now also J3.SH (SHIELD), R1.1, R2.1
- net at J2.A5 (CC1): now also R1.2
- net D+: now reaches J2.A6 (D+), J2.B6 (D+)
- net D+: now also J3.A6 (D+), J3.B6 (D+)
- net D-: now reaches J2.A7 (D-), J2.B7 (D-)
- net D-: now also J3.A7 (D-), J3.B7 (D-)
- net at J2.B5 (CC2): now also R2.2
- net VBUS: now reaches J1.A4 (VBUS), J1.A9 (VBUS), J1.B4 (VBUS), J1.B9 (VBUS), J3.A4 (VBUS), J3.A9 (VBUS), J3.B4 (VBUS), J3.B9 (VBUS)
- net CC1_POWER: now reaches J1.A5 (CC1), J3.A5 (CC1)
- net CC2_POWER: now reaches J1.B5 (CC2), J3.B5 (CC2)

Commit message: layout done, routing half way
Parts:
- J1, J2, J3: footprint Connector_USB:USB_C_Receptacle_GCT_USB4110 -> cl_Connector_USB:USB_C_Receptacle_GCT_USB4110
Changed lines of the file:
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@@
+		)
+	)
+	(netclass_flag ""
+		(length 2.54)
+		(shape round)
+		(at 133.35 71.12 0)
+		(fields_autoplaced yes)
+		(effects
+			(font
+				(size 1.27 1.27)
+			)
+			(justify left bottom)
+		)
+		(property "Netclass" "USB"
+			(at 134.0485 68.58 0)
+			(show_name no)
+			(do_not_autoplace no)
+			(effects
+				(font
+					(size 1.27 1.27)
+				)
+				(justify left)
+			)
+		)
+		(property "Component Class" ""
+			(at -1.27 0 0)
+			(show_name no)
+			(do_not_autoplace no)
+			(effects
+				(font
+					(size 1.27 1.27)
+					(italic yes)
+				)
+			)
+		)
+	)
+	(netclass_flag ""
+		(length 2.54)
+		(shape round)
+		(at 133.35 76.2 0)
+		(fields_autoplaced yes)
+		(effects
+			(font
+				(size 1.27 1.27)
+			)
+			(justify left bottom)
+		)
+		(property "Netclass" "USB"
+			(at 134.0485 73.66 0)
+			(show_name no)
+			(do_not_autoplace no)
+			(effects
+				(font
+					(size 1.27 1.27)
+				)
+				(justify left)
+			)
+		)
+		(property "Component Class" ""
+			(at -1.27 5.08 0)
+			(show_name no)
+			(do_not_autoplace no)
+			(effects
+				(font
+					(size 1.27 1.27)
+					(italic yes)
+				)
+			)
 		)
 	)
@@
 			)
 		)
-		(property "Footprint" "Connector_USB:USB_C_Receptacle_GCT_USB4110"
+		(property "Footprint" "cl_Connector_USB:USB_C_Receptacle_GCT_USB4110"
 			(at 66.04 130.81 0)
 			(hide yes)
@@
 			)
 		)
-		(property "Footprint" "Connector_USB:USB_C_Receptacle_GCT_USB4110"
+		(property "Footprint" "cl_Connector_USB:USB_C_Receptacle_GCT_USB4110"
 			(at 209.296 75.438 0)
 			(hide yes)
@@
 			)
 		)
-		(property "Footprint" "Connector_USB:USB_C_Receptacle_GCT_USB4110"
+		(property "Footprint" "cl_Connector_USB:USB_C_Receptacle_GCT_USB4110"
 			(at 66.04 71.12 0)
 			(hide yes)
